File: KiCad_Tree/LimeVR_Soda.kicad_sch (KiCad schematic)
At the start: 15 parts, among them J1 Power_IN, J2 Extension_Module, J3 UART, J4 GND, J5 CHIP_PU, J6 Power_OUT, J7 IMU_Pin_Header, U1 ESP8684-WROOM-02C

Commit message: v1.2 一个无聊又可悲的版本
我恨 esp-idf
总之，等 platformIO 支持 esp32-c2 了或许可以装上官方的固件吧
那样这些时间也不算是完全浪费
又或许 c2 和 c3 的引脚什么的都是兼容的，倒是能基本直接换掉
无聊
但也没那么无聊吧，至少让我找到了不少事情干，espidf
的文档要是写的更详细点，或许我现在也不会失去动力了吧
谁能想到所有技术栈里 freertos 和抄来的 kalmanFilter 都能弄好
最后被一个 i2c 和 spi 的驱动教训呢

这些东西感觉出现在 readme 里会更好
Parts:
- removed J4: GND, Connector_Pin:Pin_D1.0mm_L10.0mm, symbol Connector:Conn_01x01_Socket
- added J10, J11, J12, J13, J14, J16: GND_Pad, SourLemonJuice:Wire_Pad_1.5x3, symbol Connector:Conn_01x01_Socket
- added J15, J17: V5_Pad, SourLemonJuice:Wire_Pad_1.5x3, symbol Connector:Conn_01x01_Socket
- added J4: Extension_Module_2_PH-6p, Connector_JST:JST_PH_B6B-PH-K_1x06_P2.00mm_Vertical, symbol Connector:Conn_01x06_Socket
- added J8: CHIP_PU_Pinheader, Connector_PinHeader_2.54mm:PinHeader_1x02_P2.54mm_Vertical, symbol Connector:Conn_01x02_Socket
- added J9: GPIO9_Pinheader, Connector_PinHeader_2.54mm:PinHeader_1x02_P2.54mm_Vertical, symbol Connector:Conn_01x02_Pin
- C1, C2, C3, R1, R2: footprint Resistor_SMD:R_1210_3225Metric_Pad1.30x2.65mm_HandSolder -> Resistor_SMD:R_0603_1608Metric_Pad0.98x0.95mm_HandSolder
- D1: value 1N5817 -> 1N5817W; footprint Diode_THT:D_DO-41_SOD81_P7.62mm_Horizontal -> Diode_SMD:D_SOD-123
- J1: value Power_IN -> JST_PH-2p
- J2: value Extension_Module -> Extension_Module_1_PH-6p; footprint Connector_JST:JST_PH_B10B-PH-K_1x10_P2.00mm_Vertical -> Connector_JST:JST_PH_B6B-PH-K_1x06_P2.00mm_Vertical; symbol Connector:Conn_01x10_Socket -> Connector:Conn_01x06_Socket
- J3: value UART -> UART_Pinheader; footprint Connector_PinHeader_2.54mm:PinHeader_1x04_P2.54mm_Vertical -> Connector_PinHeader_2.54mm:PinHeader_1x02_P2.54mm_Vertical; symbol Connector:Conn_01x04_Pin -> Connector:Conn_01x02_Pin
- J5: value CHIP_PU -> Extension_3_pad; footprint Connector_Pin:Pin_D1.0mm_L10.0mm -> SourLemonJuice:Wire_Pad_1.5x3
- J6: value Power_OUT -> JST_PH-2p
- J7: value IMU_Pin_Header -> IMU_BMI160_Module
Connections:
- net Chip_PU: now also J8.2 (Pin_2); no longer J5.1 (Pin_1)
- net GIPO9: now also J9.2 (Pin_2); no longer J3.2 (Pin_2)
- net GND: now also J10.1 (Pin_1), J11.1 (Pin_1), J14.1 (Pin_1), J16.1 (Pin_1), J4.1 (Pin_1), J8.1 (Pin_1), J9.1 (Pin_1); no longer J3.1 (Pin_1)
- net U0RXD: now also J3.2 (Pin_2); no longer J3.4 (Pin_4)
- net U0TXD: now also J3.1 (Pin_1); no longer J3.3 (Pin_3)
- net VCC_3v3: now also J12.1 (Pin_1), J13.1 (Pin_1), J4.2 (Pin_2)
- net at D1.2 (A), J1.2 (Pin_2), J6.2 (Pin_2): now also J15.1 (Pin_1), J17.1 (Pin_1)
- net at R2.2, U1.7 (GPIO8): now also J5.1 (Pin_1)
- net at U1.18 (GPIO0/ADC1_CH0): now also J2.3 (Pin_3); no longer J2.10 (Pin_10)
- net at U1.6 (GPIO7/FSPID/MTDO): now also J4.3 (Pin_3); no longer J2.3 (Pin_3)
- net at J2.4 (Pin_4): now also U1.17 (GPIO1/ADC1_CH1); no longer U1.15 (GPIO3/ADC1_CH3)
- net at U1.5 (GPIO6/FSPICLK/MTCK): now also J4.4 (Pin_4); no longer J2.5 (Pin_5)
- net at U1.16 (GPIO1/ADC1_CH2/FSPIQ): now also J2.5 (Pin_5); no longer J2.6 (Pin_6)
- net at U1.4 (GPIO5/FSPIWP/MTDI): now also J4.5 (Pin_5); no longer J2.7 (Pin_7)
- net at U1.3 (GPIO4/ADC1_CH4/FSPIHD/MTMS): now also J4.6 (Pin_6); no longer J2.9 (Pin_9)
- new net: J2.6 (Pin_6), U1.15 (GPIO3/ADC1_CH3)
Other:
- note added: "Poser out"
- note added: "Power in"
- note removed: "ESP8684-WROOM-02C"
- title: LimeVR_Soda -> LimeVR_Soda-MCU
